File: RGBLEDController/Schematic.sch (EAGLE design)
At the start: 25 parts, among them IC1 ATMEGA168-PU, T1 TIP122, T2 TIP122, T3 TIP122, T4 TIP122

Commit message: Schematic V1.1
Parts:
- removed C1, C2, C3, C4: (no value), rcl:C-EU025-024X044
- removed C6: (no value), capacitor-wima:C2.5/2
- removed H1: MOUNT-HOLE2.8, holes:MOUNT-HOLE2.8
- removed IC1: ATMEGA168-PU, Arduino-AVR:ATMEGA168-PU
- removed IC2: (no value), v-reg:78XXS
- removed Q1: (no value), special:XTAL/S
- added LED1: DAY/NIGHT, SparkFun-LED:LED3MM
- added R5: 220, resistor:R-EU_0204/7
- added U$1: ARDUINO_PRO_MICRO, SparkFun-Boards:ARDUINO_PRO_MICRO
Connections:
- removed net N$14: IC1.DIGITAL_3(PWM), R3.2
- removed net VCC: C2.1, C6.2, IC1.VCC, IC1.VCC/ANALOG, IC2.OUT
- new net N$3: C5.+, D1.C, D2.C, D3.C, D4.C, OUTPUT-1.KL, OUTPUT-6.KL, POWER-2.KL, U$1.RAW
- net GND: now also LED1.C, U$1.GND@2; no longer C1.2, C2.2, C3.2, C4.2, C6.1, IC1.GND, IC1.GND/ANALOG, IC2.GND
- net N$1: now also LED1.A, R5.2; no longer C1.1, C5.+, D1.C, D2.C, D3.C, D4.C, IC2.IN, OUTPUT-1.KL, OUTPUT-6.KL, POWER-2.KL
- net N$13: now also R5.1, U$1.13(SCK); no longer IC1.DIGITAL_2, R4.2
- net N$15: now also U$1.*5; no longer IC1.DIGITAL_4
- net N$16: now also U$1.*3; no longer IC1.DIGITAL_5(PWM)
- net N$5: now also R4.2, U$1.*9; no longer C4.1, IC1.CRYSTAL2, Q1.2
- net N$6: now also R3.2, U$1.*6; no longer C3.1, IC1.CRYSTAL1, Q1.1
Other:
- moved on the sheet: C5, H4, POWER-1, POWER-2

Commit message: V1.2
Parts:
- T1, T2, T3, T4: value TIP122 -> (none); device transistor-neu-to92:TIP122 -> transistor:TIP122VERTICAL
Connections:
- removed net N$7: D3.A, OUTPUT-4.KL, T2.C
- removed net N$8: D2.A, OUTPUT-3.KL, T1.C
- new net N$14: D3.A, OUTPUT-4.KL, T3.C
- new net N$17: D2.A, OUTPUT-3.KL, T2.C
- net N$10: now also T3.B; no longer T2.B
- net N$11: now also T2.B; no longer T1.B
- net N$12: now also T1.B; no longer T4.B
- net N$2: now also T4.B; no longer T3.B
- net N$4: now also T4.C; no longer T3.C
- net N$9: now also T1.C; no longer T4.C
Other:
- moved on the sheet: T1, T2, T3, T4
Changed lines of the file:
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@@
 </classes>
 <parts>
-<part name="T1" library="transistor-neu-to92" deviceset="TIP122" device=""/>
-<part name="T2" library="transistor-neu-to92" deviceset="TIP122" device=""/>
-<part name="T3" library="transistor-neu-to92" deviceset="TIP122" device=""/>
-<part name="T4" library="transistor-neu-to92" deviceset="TIP122" device=""/>
 <part name="D1" library="diode" deviceset="1N4004" device=""/>
 <part name="D2" library="diode" deviceset="1N4004" device=""/>
@@
 <part name="LED1" library="SparkFun-LED" deviceset="LED" device="3MM" value="DAY/NIGHT"/>
 <part name="R5" library="resistor" deviceset="R-EU_" device="0204/7" value="220"/>
+<part name="T1" library="transistor" deviceset="TIP122" device="VERTICAL"/>
+<part name="T2" library="transistor" deviceset="TIP122" device="VERTICAL"/>
+<part name="T3" library="transistor" deviceset="TIP122" device="VERTICAL"/>
+<part name="T4" library="transistor" deviceset="TIP122" device="VERTICAL"/>
 </parts>
 <sheets>
@@
 </plain>
 <instances>
-<instance part="T1" gate="G$1" x="55.88" y="58.42" rot="R180"/>
-<instance part="T2" gate="G$1" x="55.88" y="43.18" rot="R180"/>
-<instance part="T3" gate="G$1" x="55.88" y="27.94" rot="R180"/>
-<instance part="T4" gate="G$1" x="55.88" y="73.66" rot="R180"/>
 <instance part="D1" gate="1" x="20.32" y="76.2" rot="R90"/>
 <instance part="D2" gate="1" x="20.32" y="60.96" rot="R90"/>
@@
 <instance part="LED1" gate="G$1" x="121.92" y="38.1" rot="R90"/>
 <instance part="R5" gate="G$1" x="111.76" y="38.1"/>
+<instance part="T1" gate="G$1" x="55.88" y="73.66" rot="R180"/>
+<instance part="T2" gate="G$1" x="55.88" y="58.42" rot="R180"/>
+<instance part="T3" gate="G$1" x="55.88" y="43.18" rot="R180"/>
+<instance part="T4" gate="G$1" x="55.88" y="27.94" rot="R180"/>
 </instances>
 <busses>
@@
 <segment>
 <pinref part="GND3" gate="1" pin="GND"/>
+<wire x1="50.8" y1="81.28" x2="48.26" y2="81.28" width="0.1524" layer="91"/>
+<pinref part="T1" gate="G$1" pin="E"/>
+</segment>
+<segment>
+<pinref part="GND4" gate="1" pin="GND"/>
+<wire x1="48.26" y1="66.04" x2="50.8" y2="66.04" width="0.1524" layer="91"/>
+<pinref part="T2" gate="G$1" pin="E"/>
+</segment>
+<segment>
+<pinref part="GND5" gate="1" pin="GND"/>
+<wire x1="48.26" y1="50.8" x2="50.8" y2="50.8" width="0.1524" layer="91"/>
+<pinref part="T3" gate="G$1" pin="E"/>
+</segment>
+<segment>
+<pinref part="GND6" gate="1" pin="GND"/>
+<wire x1="48.26" y1="35.56" x2="50.8" y2="35.56" width="0.1524" layer="91"/>
 <pinref part="T4" gate="G$1" pin="E"/>
-<wire x1="50.8" y1="81.28" x2="48.26" y2="81.28" width="0.1524" layer="91"/>
-</segment>
-<segment>
-<pinref part="GND4" gate="1" pin="GND"/>
-<pinref part="T1" gate="G$1" pin="E"/>
-<wire x1="48.26" y1="66.04" x2="50.8" y2="66.04" width="0.1524" layer="91"/>
-</segment>
-<segment>
-<pinref part="GND5" gate="1" pin="GND"/>
-<pinref part="T2" gate="G$1" pin="E"/>
-<wire x1="48.26" y1="50.8" x2="50.8" y2="50.8" width="0.1524" layer="91"/>
-<junction x="50.8" y="50.8"/>
-</segment>
-<segment>
-<pinref part="GND6" gate="1" pin="GND"/>
-<pinref part="T3" gate="G$1" pin="E"/>
-<wire x1="48.26" y1="35.56" x2="50.8" y2="35.56" width="0.1524" layer="91"/>
 </segment>
 <segment>
@@
 <wire x1="17.78" y1="25.4" x2="20.32" y2="25.4" width="0.1524" layer="91"/>
 <wire x1="20.32" y1="25.4" x2="20.32" y2="22.86" width="0.1524" layer="91"/>
-<pinref part="T3" gate="G$1" pin="C"/>
 <junction x="20.32" y="25.4"/>
 <wire x1="20.32" y1="25.4" x2="50.8" y2="25.4" width="0.1524" layer="91"/>
-</segment>
-</net>
-<net name="N$7" class="0">
+<pinref part="T4" gate="G$1" pin="C"/>
+</segment>
+</net>
+<net name="N$14" class="0">
 <segment>
 <pinref part="OUTPUT" gate="-4" pin="KL"/>
@@
 <wire x1="17.78" y1="40.64" x2="20.32" y2="40.64" width="0.1524" layer="91"/>
 <wire x1="20.32" y1="40.64" x2="20.32" y2="38.1" width="0.1524" layer="91"/>
-<pinref part="T2" gate="G$1" pin="C"/>
 <junction x="20.32" y="40.64"/>
 <wire x1="20.32" y1="40.64" x2="50.8" y2="40.64" width="0.1524" layer="91"/>
-</segment>
-</net>
-<net name="N$8" class="0">
+<pinref part="T3" gate="G$1" pin="C"/>
+</segment>
+</net>
+<net name="N$17" class="0">
 <segment>
 <pinref part="OUTPUT" gate="-3" pin="KL"/>
@@
 <wire x1="17.78" y1="55.88" x2="20.32" y2="55.88" width="0.1524" layer="91"/>
 <wire x1="20.32" y1="55.88" x2="20.32" y2="58.42" width="0.1524" layer="91"/>
-<pinref part="T1" gate="G$1" pin="C"/>
 <junction x="20.32" y="55.88"/>
 <wire x1="20.32" y1="55.88" x2="50.8" y2="55.88" width="0.1524" layer="91"/>
+<pinref part="T2" gate="G$1" pin="C"/>
 </segment>
 </net>
@@
 <wire x1="17.78" y1="71.12" x2="20.32" y2="71.12" width="0.1524" layer="91"/>
 <wire x1="20.32" y1="71.12" x2="20.32" y2="73.66" width="0.1524" layer="91"/>
-<pinref part="T4" gate="G$1" pin="C"/>
 <junction x="20.32" y="71.12"/>
 <wire x1="20.32" y1="71.12" x2="50.8" y2="71.12" width="0.1524" layer="91"/>
+<pinref part="T1" gate="G$1" pin="C"/>
 </segment>
 </net>
 <net name="N$2" class="0">
 <segment>
-<pinref part="T3" gate="G$1" pin="B"/>
 <pinref part="R4" gate="G$1" pin="1"/>
 <wire x1="58.42" y1="27.94" x2="60.96" y2="27.94" width="0.1524" layer="91"/>
+<pinref part="T4" gate="G$1" pin="B"/>
 </segment>
 </net>
 <net name="N$10" class="0">
 <segment>
-<pinref part="T2" gate="G$1" pin="B"/>
 <pinref part="R3" gate="G$1" pin="1"/>
 <wire x1="58.42" y1="43.18" x2="60.96" y2="43.18" width="0.1524" layer="91"/>
+<pinref part="T3" gate="G$1" pin="B"/>
 </segment>
 </net>
 <net name="N$11" class="0">
 <segment>
-<pinref part="T1" gate="G$1" pin="B"/>
 <pinref part="R2" gate="G$1" pin="1"/>
 <wire x1="58.42" y1="58.42" x2="60.96" y2="58.42" width="0.1524" layer="91"/>
+<pinref part="T2" gate="G$1" pin="B"/>
 </segment>
 </net>
 <net name="N$12" class="0">
 <segment>
-<pinref part="T4" gate="G$1" pin="B"/>
 <pinref part="R1" gate="G$1" pin="1"/>
 <wire x1="58.42" y1="73.66" x2="60.96" y2="73.66" width="0.1524" layer="91"/>
-</segment>
-</net>
+<pinref part="T1" gate="G$1" pin="B"/>
+</segment>
+</net>
